File: kicad/OnGod.kicad_sch (KiCad schematic)
At the start: 16 parts, among them J1 Speaker, J2 Servo, J3 Servo, J4 Servo, J5 Servo, J6 7.4LipoXT30, J7 HM10-Bluetooth, J8 7.4LipoXT30, J9 Servo, M1 N20Motor_DC, M2 N20Motor_DC, U1 XIAO-ESP32-C3-DIP, U2 H-BridgeDRV8833PW, U4 BuckConverterR-78E5.0-1.0

Commit message: updated schematic
Parts:
- removed R1, R2: 10k, symbol Device:R
- added C1: 0.1uF, symbol Device:C
- added R3: 10k, symbol Device:R
- added SW1: SW_SPST, symbol Switch:SW_SPST
Connections:
- net +5V: now also U2.12 (VM), U4.3 (OUT), C1.1, SW1.1 (A)
- net GND: now also J6.2 (Pin_2), U1.13 (GND), U2.13 (GND), U2.3 (AISEN), U2.6 (BISEN), U4.2 (GND)
- net BatteryPower: now reaches J6.1 (Pin_1)
- net BatteryPower: now also U4.1 (IN)
- net Sleep: now reaches U2.1 (~{SLEEP})
- net Sleep: now also U1.11 (GPIO10/D10/MOSI)
- net RightDriveIn2: now reaches U2.10 (BIN2)
- net RightDriveIn2: now also U1.4 (GPIO5/A3/D3)
- net at U2.11 (VCP): now also C1.2
- net LeftDriveIn1: now reaches U2.15 (AIN2)
- net LeftDriveIn1: now also U1.1 (GPIO2/A0/D0), U1.2 (GPIO3/A1/D1), U1.3 (GPIO4/A2/D2), U2.16 (AIN1), U2.9 (BIN1)
- net LeftDriveOut1: now reaches U2.2 (AOUT1)
- net LeftDriveOut1: now also M1.1 (+)
- net LeftDriveOut2: now reaches U2.4 (AOUT2)
- net LeftDriveOut2: now also M1.2 (-)
- net RightDriveOut2: now reaches U2.5 (BOUT2)
- net RightDriveOut2: now also M2.2 (-)
- net RightDriveOut1: now reaches U2.7 (BOUT1)
- net RightDriveOut1: now also M2.1 (+)
- net at U2.8 (~{FAULT}): now also R3.1
- net +3V3: now reaches U1.12 (VCC_3V3)
- net +3V3: now also R3.2
- net VBUS: now reaches U1.14 (VBUS)
- net VBUS: now also SW1.2 (B)
Other:
- moved on the sheet: J1, J2, J3, J4, J5, J8, J9, M1, M2, U2, U4
